Commit message: Fix drone spawning using absolute paths

File: RLDrone/aero_control/models/aero/intel_aero.xacro (robot description, xacro)
@@ -5,5 +5,5 @@
   <xacro:property name="rotor_velocity_slowdown_sim" value="10" />
   <xacro:property name="use_mesh_file" value="true" />
-  <xacro:property name="mesh_file" value="package://rotors_description/meshes/intel_aero.dae" />
+  <xacro:property name="mesh_file" value="./meshes/intel_aero.dae" />
   <xacro:property name="mass" value="1.2" /> <!-- [kg] -->
   <xacro:property name="body_width" value="0.285" /> <!-- [m] -->
@@ -34,5 +34,5 @@
     </xacro:property>
     <!-- Included URDF Files -->
-    <xacro:include filename="$(find rotors_description)/urdf/multirotor_base.xacro" />
+    <xacro:include filename="$(find aero_control)/models/aero/multirotor_base.xacro" />
     <!-- Instantiate multirotor_base_macro once -->
     <xacro:multirotor_base_macro
@@ -64,5 +64,5 @@
       color="Red"
       use_own_mesh="true"
-      mesh="package://rotors_description/meshes/intel_aero_propeller.dae">
+      mesh="./meshes/intel_aero_propeller.dae">
       <origin xyz="${arm_length / sqrt2} -${arm_length / sqrt2} ${rotor_offset_top}" rpy="0 0 0" />
       <xacro:insert_block name="rotor_inertia" />
@@ -85,5 +85,5 @@
       color="Blue"
       use_own_mesh="true"
-      mesh="package://rotors_description/meshes/intel_aero_propeller.dae">
+      mesh="./meshes/intel_aero_propeller.dae">
       <origin xyz="-${arm_length / sqrt2} ${arm_length / sqrt2} ${rotor_offset_top}" rpy="0 0 0" />
       <xacro:insert_block name="rotor_inertia" />
@@ -105,5 +105,5 @@
       color="Red"
       use_own_mesh="true"
-      mesh="package://rotors_description/meshes/intel_aero_propeller.dae">
+      mesh="./meshes/intel_aero_propeller.dae">
       <origin xyz="${arm_length / sqrt2} ${arm_length / sqrt2} ${rotor_offset_top}" rpy="0 0 0" />
       <xacro:insert_block name="rotor_inertia" />
@@ -125,5 +125,5 @@
       color="Blue"
       use_own_mesh="true"
-      mesh="package://rotors_description/meshes/intel_aero_propeller.dae">
+      mesh="./meshes/intel_aero_propeller.dae">
       <origin xyz="-${arm_length / sqrt2} -${arm_length / sqrt2} ${rotor_offset_top}" rpy="0 0 0" />
       <xacro:insert_block name="rotor_inertia" />

File: RLDrone/aero_control/models/aero/intel_aero_base.xacro (robot description, xacro)
@@ -1,7 +1,7 @@
 <?xml version="1.0"?>
 <robot name="aero" xmlns:xacro="http://ros.org/wiki/xacro">
-  <xacro:include filename="$(find rotors_description)/urdf/component_snippets.xacro" />
+  <xacro:include filename="$(find aero_control)/models/aero/component_snippets.xacro" />
   <!-- Instantiate ardrone "mechanics" -->
-  <xacro:include filename="$(find rotors_description)/urdf/intel_aero.xacro" />
+  <xacro:include filename="$(find aero_control)/models/aero/intel_aero.xacro" />
   <!-- Instantiate a controller. -->
   <xacro:controller_plugin_macro namespace="${namespace}" imu_sub_topic="imu" />
